File: TeensySonarBoard.brd (EAGLE design)
At the start: 59.7 x 53.3 mm, 10 parts, among them J5 RJ45, U1 MIC5219 3.3V

Commit message: Changed design rules to gold pheonix.
Routing:
- net Z: track 24.0 -> 14.6 mm, vias 0 -> 1
- net Y: track 17.9 -> 15.8 mm
Changed lines of the file:
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@@
 </class>
 </classes>
-<designrules name="OSHpark">
-<description language="de">&lt;b&gt;EAGLE Design Rules&lt;/b&gt;
+<designrules name="GoldPhoenix">
+<description language="en">
+&lt;b&gt;Gold Phoenix PCB Design Rules&lt;/b&gt;
 &lt;p&gt;
-Die Standard-Design-Rules sind so gewählt, dass sie für
-die meisten Anwendungen passen. Sollte ihre Platine
-besondere Anforderungen haben, treffen Sie die erforderlichen
-Einstellungen hier und speichern die Design Rules unter
-einem neuen Namen ab.</description>
-<description language="en">&lt;b&gt;Laen's PCB Order Design Rules&lt;/b&gt;
-&lt;p&gt;
-Please make sure your boards conform to these design rules.</description>
+Created by Nick Molo for the Purdue IEEE ROV Team
+</description>
 <param name="layerSetup" value="(1*16)"/>
-<param name="mtCopper" value="0.0356mm 0.0356mm 0.0356mm 0.0356mm 0.0356mm 0.0356mm 0.0356mm 0.0356mm 0.0356mm 0.0356mm 0.0356mm 0.0356mm 0.0356mm 0.0356mm 0.0356mm 0.0356mm"/>
-<param name="mtIsolate" value="1.5011mm 0.1499mm 0.2007mm 0.1499mm 0.2007mm 0.1499mm 0.2007mm 0.1499mm 0.2007mm 0.1499mm 0.2007mm 0.1499mm 0.2007mm 0.1499mm 0.2007mm"/>
-<param name="mdWireWire" value="6mil"/>
-<param name="mdWirePad" value="6mil"/>
-<param name="mdWireVia" value="6mil"/>
-<param name="mdPadPad" value="6mil"/>
-<param name="mdPadVia" value="6mil"/>
-<param name="mdViaVia" value="6mil"/>
-<param name="mdSmdPad" value="6mil"/>
-<param name="mdSmdVia" value="6mil"/>
-<param name="mdSmdSmd" value="6mil"/>
+<param name="mtCopper" value="0.035mm 0.035mm 0.035mm 0.035mm 0.035mm 0.035mm 0.035mm 0.035mm 0.035mm 0.035mm 0.035mm 0.035mm 0.035mm 0.035mm 0.035mm 0.035mm"/>
+<param name="mtIsolate" value="1.5mm 0.15mm 0.2mm 0.15mm 0.2mm 0.15mm 0.2mm 0.15mm 0.2mm 0.15mm 0.2mm 0.15mm 0.2mm 0.15mm 0.2mm"/>
+<param name="mdWireWire" value="7mil"/>
+<param name="mdWirePad" value="7mil"/>
+<param name="mdWireVia" value="7mil"/>
+<param name="mdPadPad" value="7mil"/>
+<param name="mdPadVia" value="7mil"/>
+<param name="mdViaVia" value="7mil"/>
+<param name="mdSmdPad" value="7mil"/>
+<param name="mdSmdVia" value="7mil"/>
+<param name="mdSmdSmd" value="7mil"/>
 <param name="mdViaViaSameLayer" value="8mil"/>
 <param name="mnLayersViaInSmd" value="2"/>
-<param name="mdCopperDimension" value="15mil"/>
-<param name="mdDrill" value="6mil"/>
+<param name="mdCopperDimension" value="10mil"/>
+<param name="mdDrill" value="8mil"/>
 <param name="mdSmdStop" value="0mil"/>
-<param name="msWidth" value="6mil"/>
-<param name="msDrill" value="13mil"/>
-<param name="msMicroVia" value="13mil"/>
+<param name="msWidth" value="7mil"/>
+<param name="msDrill" value="10mil"/>
+<param name="msMicroVia" value="9.99mm"/>
 <param name="msBlindViaRatio" value="0.5"/>
 <param name="rvPadTop" value="0.25"/>
@@
 <param name="rvMicroViaOuter" value="0.25"/>
 <param name="rvMicroViaInner" value="0.25"/>
-<param name="rlMinPadTop" value="7mil"/>
+<param name="rlMinPadTop" value="10mil"/>
 <param name="rlMaxPadTop" value="20mil"/>
-<param name="rlMinPadInner" value="7mil"/>
+<param name="rlMinPadInner" value="10mil"/>
 <param name="rlMaxPadInner" value="20mil"/>
-<param name="rlMinPadBottom" value="7mil"/>
+<param name="rlMinPadBottom" value="10mil"/>
 <param name="rlMaxPadBottom" value="20mil"/>
-<param name="rlMinViaOuter" value="7mil"/>
+<param name="rlMinViaOuter" value="10mil"/>
 <param name="rlMaxViaOuter" value="20mil"/>
-<param name="rlMinViaInner" value="7mil"/>
+<param name="rlMinViaInner" value="10mil"/>
 <param name="rlMaxViaInner" value="20mil"/>
 <param name="rlMinMicroViaOuter" value="4mil"/>
@@
 <param name="mvStopFrame" value="1"/>
 <param name="mvCreamFrame" value="0"/>
-<param name="mlMinStopFrame" value="3mil"/>
-<param name="mlMaxStopFrame" value="3mil"/>
+<param name="mlMinStopFrame" value="4mil"/>
+<param name="mlMaxStopFrame" value="4mil"/>
 <param name="mlMinCreamFrame" value="0mil"/>
 <param name="mlMaxCreamFrame" value="0mil"/>
-<param name="mlViaStopLimit" value="0mil"/>
+<param name="mlViaStopLimit" value="25mil"/>
 <param name="srRoundness" value="0"/>
 <param name="srMinRoundness" value="0mil"/>
@@
 </elements>
 <signals>
-<signal name="GND">
+<signal name="GND" airwireshidden="yes">
 <contactref element="U1" pad="2"/>
 <contactref element="C1" pad="2"/>
@@
 <wire x1="20.32" y1="20.32" x2="21.59" y2="19.05" width="0.4064" layer="1"/>
 <wire x1="21.59" y1="19.05" x2="21.59" y2="18.63" width="0.4064" layer="1"/>
-<wire x1="3.81" y1="41.91" x2="3.81" y2="43.18" width="0.3048" layer="16"/>
-<wire x1="3.81" y1="43.18" x2="5.08" y2="44.45" width="0.3048" layer="16"/>
-<wire x1="5.08" y1="44.45" x2="29.21" y2="44.45" width="0.3048" layer="16"/>
-<wire x1="29.21" y1="44.45" x2="33.02" y2="48.26" width="0.3048" layer="16"/>
-<wire x1="33.02" y1="48.26" x2="33.02" y2="50.8" width="0.3048" layer="16"/>
+<wire x1="3.81" y1="41.91" x2="3.81" y2="43.18" width="0.4064" layer="16"/>
+<wire x1="3.81" y1="43.18" x2="5.08" y2="44.45" width="0.4064" layer="16"/>
+<wire x1="5.08" y1="44.45" x2="29.21" y2="44.45" width="0.4064" layer="16"/>
+<wire x1="29.21" y1="44.45" x2="33.02" y2="48.26" width="0.4064" layer="16"/>
+<wire x1="33.02" y1="48.26" x2="33.02" y2="50.8" width="0.4064" layer="16"/>
 <contactref element="U$1" pad="VCC13"/>
 <contactref element="U$1" pad="VCC14"/>
@@
 <contactref element="U$1" pad="Y"/>
 <contactref element="J5" pad="8"/>
-<wire x1="42.7485" y1="12.7" x2="40.64" y2="12.7" width="0.3048" layer="1"/>
-<wire x1="40.64" y1="12.7" x2="39.37" y2="13.97" width="0.3048" layer="1"/>
-<via x="39.37" y="13.97" extent="1-16" drill="0.6"/>
-<wire x1="39.37" y1="13.97" x2="39.37" y2="17.78" width="0.3048" layer="16"/>
-<wire x1="39.37" y1="17.78" x2="41.91" y2="20.32" width="0.3048" layer="16"/>
-<wire x1="41.91" y1="20.32" x2="47.625" y2="20.32" width="0.3048" layer="16"/>
-<wire x1="47.625" y1="20.32" x2="48.26" y2="19.685" width="0.3048" layer="16"/>
+<wire x1="42.7485" y1="12.7" x2="41.275" y2="12.7" width="0.3048" layer="1"/>
+<wire x1="41.275" y1="12.7" x2="40.767" y2="13.208" width="0.3048" layer="1"/>
+<wire x1="40.767" y1="13.208" x2="40.767" y2="16.891" width="0.3048" layer="1"/>
+<via x="40.767" y="16.891" extent="1-16" drill="0.6"/>
+<wire x1="40.767" y1="16.891" x2="40.767" y2="19.05" width="0.3048" layer="16"/>
+<wire x1="40.767" y1="19.05" x2="41.402" y2="19.685" width="0.3048" layer="16"/>
+<wire x1="41.402" y1="19.685" x2="48.26" y2="19.685" width="0.3048" layer="16"/>
 </signal>
 <signal name="Z">
 <contactref element="U$1" pad="Z"/>
 <contactref element="J5" pad="7"/>
-<wire x1="42.7485" y1="13.97" x2="44.45" y2="13.97" width="0.3048" layer="1"/>
-<wire x1="44.45" y1="13.97" x2="45.72" y2="12.7" width="0.3048" layer="1"/>
-<wire x1="45.72" y1="12.7" x2="45.72" y2="10.16" width="0.3048" layer="1"/>
-<wire x1="45.72" y1="10.16" x2="46.99" y2="8.89" width="0.3048" layer="1"/>
-<wire x1="46.99" y1="8.89" x2="52.07" y2="8.89" width="0.3048" layer="1"/>
-<wire x1="52.07" y1="8.89" x2="53.34" y2="10.16" width="0.3048" layer="1"/>
-<wire x1="53.34" y1="10.16" x2="53.34" y2="15.875" width="0.3048" layer="1"/>
-<wire x1="53.34" y1="15.875" x2="50.8" y2="18.415" width="0.3048" layer="1"/>
+<wire x1="44.45" y1="18.542" x2="44.704" y2="18.796" width="0.3048" layer="16"/>
+<wire x1="44.704" y1="18.796" x2="46.736" y2="18.796" width="0.3048" layer="16"/>
+<wire x1="46.736" y1="18.796" x2="47.117" y2="18.415" width="0.3048" layer="16"/>
+<wire x1="47.117" y1="18.415" x2="50.8" y2="18.415" width="0.3048" layer="16"/>
+<wire x1="44.45" y1="18.542" x2="44.45" y2="15.621" width="0.3048" layer="16"/>
+<wire x1="44.45" y1="15.621" x2="45.72" y2="14.351" width="0.3048" layer="16"/>
+<via x="45.72" y="14.351" extent="1-16" drill="0.6"/>
+<wire x1="45.72" y1="14.351" x2="45.72" y2="14.097" width="0.3048" layer="1"/>
+<wire x1="45.72" y1="14.097" x2="45.593" y2="13.97" width="0.3048" layer="1"/>
+<wire x1="45.593" y1="13.97" x2="42.7485" y2="13.97" width="0.3048" layer="1"/>
 </signal>
 <signal name="A0">

Commit message: Added a 2A fuse to the board to meet MATE requirements.
Parts:
- added F1: 2A, MotherboardParts:KEYSTONE_FUSE_3587
Connections:
- new net N$1: BATT.2, F1.P$1, F1.P$2
- net VCC: now also F1.P$3, F1.P$4; no longer BATT.2
Routing:
- net VCC: track 16.7 -> 32.2 mm
- net N$1: track 0.00 -> 15.4 mm
Changed lines of the file:
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@@
 </class>
 </classes>
-<designrules name="GoldPhoenix">
-<description language="en">
-&lt;b&gt;Gold Phoenix PCB Design Rules&lt;/b&gt;
+<designrules name="OSHpark">
+<description language="de">&lt;b&gt;EAGLE Design Rules&lt;/b&gt;
 &lt;p&gt;
-Created by Nick Molo for the Purdue IEEE ROV Team
-</description>
+Die Standard-Design-Rules sind so gewählt, dass sie für
+die meisten Anwendungen passen. Sollte ihre Platine
+besondere Anforderungen haben, treffen Sie die erforderlichen
+Einstellungen hier und speichern die Design Rules unter
+einem neuen Namen ab.</description>
+<description language="en">&lt;b&gt;Laen's PCB Order Design Rules&lt;/b&gt;
+&lt;p&gt;
+Please make sure your boards conform to these design rules.</description>
 <param name="layerSetup" value="(1*16)"/>
-<param name="mtCopper" value="0.035mm 0.035mm 0.035mm 0.035mm 0.035mm 0.035mm 0.035mm 0.035mm 0.035mm 0.035mm 0.035mm 0.035mm 0.035mm 0.035mm 0.035mm 0.035mm"/>
-<param name="mtIsolate" value="1.5mm 0.15mm 0.2mm 0.15mm 0.2mm 0.15mm 0.2mm 0.15mm 0.2mm 0.15mm 0.2mm 0.15mm 0.2mm 0.15mm 0.2mm"/>
-<param name="mdWireWire" value="7mil"/>
-<param name="mdWirePad" value="7mil"/>
-<param name="mdWireVia" value="7mil"/>
-<param name="mdPadPad" value="7mil"/>
-<param name="mdPadVia" value="7mil"/>
-<param name="mdViaVia" value="7mil"/>
-<param name="mdSmdPad" value="7mil"/>
-<param name="mdSmdVia" value="7mil"/>
-<param name="mdSmdSmd" value="7mil"/>
+<param name="mtCopper" value="0.0356mm 0.0356mm 0.0356mm 0.0356mm 0.0356mm 0.0356mm 0.0356mm 0.0356mm 0.0356mm 0.0356mm 0.0356mm 0.0356mm 0.0356mm 0.0356mm 0.0356mm 0.0356mm"/>
+<param name="mtIsolate" value="1.5011mm 0.1499mm 0.2007mm 0.1499mm 0.2007mm 0.1499mm 0.2007mm 0.1499mm 0.2007mm 0.1499mm 0.2007mm 0.1499mm 0.2007mm 0.1499mm 0.2007mm"/>
+<param name="mdWireWire" value="6mil"/>
+<param name="mdWirePad" value="6mil"/>
+<param name="mdWireVia" value="6mil"/>
+<param name="mdPadPad" value="6mil"/>
+<param name="mdPadVia" value="6mil"/>
+<param name="mdViaVia" value="6mil"/>
+<param name="mdSmdPad" value="6mil"/>
+<param name="mdSmdVia" value="6mil"/>
+<param name="mdSmdSmd" value="6mil"/>
 <param name="mdViaViaSameLayer" value="8mil"/>
 <param name="mnLayersViaInSmd" value="2"/>
-<param name="mdCopperDimension" value="10mil"/>
-<param name="mdDrill" value="8mil"/>
+<param name="mdCopperDimension" value="15mil"/>
+<param name="mdDrill" value="6mil"/>
 <param name="mdSmdStop" value="0mil"/>
-<param name="msWidth" value="7mil"/>
-<param name="msDrill" value="10mil"/>
-<param name="msMicroVia" value="9.99mm"/>
+<param name="msWidth" value="6mil"/>
+<param name="msDrill" value="13mil"/>
+<param name="msMicroVia" value="13mil"/>
 <param name="msBlindViaRatio" value="0.5"/>
 <param name="rvPadTop" value="0.25"/>
@@
 <param name="rvMicroViaOuter" value="0.25"/>
 <param name="rvMicroViaInner" value="0.25"/>
-<param name="rlMinPadTop" value="10mil"/>
+<param name="rlMinPadTop" value="7mil"/>
 <param name="rlMaxPadTop" value="20mil"/>
-<param name="rlMinPadInner" value="10mil"/>
+<param name="rlMinPadInner" value="7mil"/>
 <param name="rlMaxPadInner" value="20mil"/>
-<param name="rlMinPadBottom" value="10mil"/>
+<param name="rlMinPadBottom" value="7mil"/>
 <param name="rlMaxPadBottom" value="20mil"/>
-<param name="rlMinViaOuter" value="10mil"/>
+<param name="rlMinViaOuter" value="7mil"/>
 <param name="rlMaxViaOuter" value="20mil"/>
-<param name="rlMinViaInner" value="10mil"/>
+<param name="rlMinViaInner" value="7mil"/>
 <param name="rlMaxViaInner" value="20mil"/>
 <param name="rlMinMicroViaOuter" value="4mil"/>
@@
 <param name="mvStopFrame" value="1"/>
 <param name="mvCreamFrame" value="0"/>
-<param name="mlMinStopFrame" value="4mil"/>
-<param name="mlMaxStopFrame" value="4mil"/>
+<param name="mlMinStopFrame" value="3mil"/>
+<param name="mlMaxStopFrame" value="3mil"/>
 <param name="mlMinCreamFrame" value="0mil"/>
 <param name="mlMaxCreamFrame" value="0mil"/>
-<param name="mlViaStopLimit" value="25mil"/>
+<param name="mlViaStopLimit" value="0mil"/>
 <param name="srRoundness" value="0"/>
 <param name="srMinRoundness" value="0mil"/>
@@
 </element>
 <element name="U$1" library="BackplaneParts" package="MAX3491" value="MAX3491" x="36.83" y="11.43"/>
+<element name="F1" library="MotherboardParts" package="KEYSTONE_FUSE_3587" value="2A" x="16.51" y="10.16"/>
 </elements>
 <signals>
@@
 <contactref element="U1" pad="1"/>
 <contactref element="C1" pad="1"/>
-<contactref element="BATT" pad="2"/>
 <contactref element="U1" pad="3"/>
-<wire x1="4.36" y1="18.78" x2="12.55" y2="18.78" width="0.4064" layer="1"/>
 <wire x1="12.55" y1="18.78" x2="12.7" y2="18.63" width="0.4064" layer="1"/>
 <wire x1="12.7" y1="18.63" x2="16.3799" y2="18.63" width="0.4064" layer="1"/>
@@
 <wire x1="16.4799" y1="16.83" x2="14.5" y2="16.83" width="0.4064" layer="1"/>
 <wire x1="14.5" y1="16.83" x2="12.7" y2="18.63" width="0.4064" layer="1"/>
+<contactref element="F1" pad="P$4"/>
+<contactref element="F1" pad="P$3"/>
+<wire x1="23.241" y1="7.1247" x2="23.241" y2="13.1953" width="0.4064" layer="1"/>
+<wire x1="23.241" y1="13.1953" x2="13.7287" y2="13.1953" width="0.4064" layer="1"/>
+<wire x1="13.7287" y1="13.1953" x2="10.922" y2="16.002" width="0.4064" layer="1"/>
+<wire x1="10.922" y1="16.002" x2="10.922" y2="18.034" width="0.4064" layer="1"/>
+<wire x1="10.922" y1="18.034" x2="11.43" y2="18.542" width="0.4064" layer="1"/>
+<wire x1="11.43" y1="18.542" x2="12.612" y2="18.542" width="0.4064" layer="1"/>
+<wire x1="12.612" y1="18.542" x2="12.7" y2="18.63" width="0.4064" layer="1"/>
 </signal>
 <signal name="3.3V">
@@
 <wire x1="16.51" y1="24.13" x2="13.97" y2="26.67" width="0.3048" layer="1"/>
 </signal>
+<signal name="N$1">
+<contactref element="BATT" pad="2"/>
+<contactref element="F1" pad="P$2"/>
+<contactref element="F1" pad="P$1"/>
+<wire x1="9.779" y1="7.1247" x2="9.779" y2="13.1953" width="0.4064" layer="1"/>
+<wire x1="9.779" y1="13.1953" x2="9.779" y2="15.875" width="0.4064" layer="1"/>
+<wire x1="9.779" y1="15.875" x2="6.858" y2="18.796" width="0.4064" layer="1"/>
+<wire x1="6.858" y1="18.796" x2="4.376" y2="18.796" width="0.4064" layer="1"/>
+<wire x1="4.376" y1="18.796" x2="4.36" y2="18.78" width="0.4064" layer="1"/>
+</signal>
 </signals>
