File: TeensySonarBoard.brd (EAGLE design)
At the start: 59.7 x 53.3 mm, 11 parts, among them J5 RJ45, U1 MIC5219 3.3V

Commit message: Initial placement of diagnostic LEDs.
Parts:
- added D1, D2, D3, D4, D5: (no value), SparkFun-LED:LED-0603
Connections:
- new net N$2: D5.A, TEENSY2.7
- new net N$3: D4.A, TEENSY2.9
- new net N$4: D3.A, TEENSY2.11
- new net N$5: D1.A, F1.P$3, F1.P$4
- new net N$6: C2.1, D2.A, U1.5
- net 3.3V: now also D2.C; no longer C2.1, U1.5
- net GND: now also D3.C, D4.C, D5.C
- net VCC: now also D1.C; no longer F1.P$3, F1.P$4
Routing:
- net VCC: track 32.2 -> 16.6 mm
- net 3.3V: track 106.7 -> 102.0 mm
- net N$6: track 0.00 -> 2.55 mm
Changed lines of the file:
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@@
 <element name="U$1" library="BackplaneParts" package="MAX3491" value="MAX3491" x="36.83" y="11.43"/>
 <element name="F1" library="MotherboardParts" package="KEYSTONE_FUSE_3587" value="2A" x="16.51" y="10.16"/>
+<element name="D1" library="SparkFun-LED" package="LED-0603" value="" x="-3.81" y="-10.16"/>
+<element name="D2" library="SparkFun-LED" package="LED-0603" value="" x="-3.81" y="-13.97"/>
+<element name="D3" library="SparkFun-LED" package="LED-0603" value="" x="-3.81" y="-17.78"/>
+<element name="D4" library="SparkFun-LED" package="LED-0603" value="" x="-3.81" y="-21.59"/>
+<element name="D5" library="SparkFun-LED" package="LED-0603" value="" x="-3.81" y="-25.4"/>
 </elements>
 <signals>
@@
 <vertex x="59.69" y="0"/>
 </polygon>
+<contactref element="D5" pad="C"/>
+<contactref element="D4" pad="C"/>
+<contactref element="D3" pad="C"/>
+<wire x1="27.94" y1="50.8" x2="39.37" y2="41.91" width="0" layer="19" extent="1-1"/>
+<wire x1="25.4" y1="50.8" x2="27.94" y2="50.8" width="0" layer="19" extent="1-1"/>
+<wire x1="6.35" y1="41.91" x2="25.4" y2="50.8" width="0" layer="19" extent="1-1"/>
+<wire x1="3.81" y1="26.67" x2="6.35" y2="41.91" width="0" layer="19" extent="1-1"/>
+<wire x1="4.36" y1="16.78" x2="3.81" y2="26.67" width="0" layer="19" extent="1-1"/>
+<wire x1="12.7" y1="16.93" x2="4.36" y2="16.78" width="0" layer="19" extent="1-1"/>
+<wire x1="16.4799" y1="17.78" x2="12.7" y2="16.93" width="0" layer="19" extent="1-1"/>
+<wire x1="21.59" y1="16.93" x2="16.4799" y2="17.78" width="0" layer="19" extent="1-1"/>
+<wire x1="36.83" y1="12.7" x2="21.59" y2="16.93" width="0" layer="19" extent="1-1"/>
+<wire x1="36.83" y1="11.43" x2="36.83" y2="12.7" width="0" layer="19" extent="1-1"/>
+<wire x1="41.91" y1="2.54" x2="36.83" y2="11.43" width="0" layer="19" extent="1-1"/>
+<wire x1="-3.81" y1="-16.903" x2="4.36" y2="16.78" width="0" layer="19" extent="1-1"/>
+<wire x1="-3.81" y1="-20.713" x2="-3.81" y2="-16.903" width="0" layer="19" extent="1-1"/>
+<wire x1="-3.81" y1="-24.523" x2="-3.81" y2="-20.713" width="0" layer="19" extent="1-1"/>
 </signal>
 <signal name="VCC">
@@
 <wire x1="16.4799" y1="16.83" x2="14.5" y2="16.83" width="0.4064" layer="1"/>
 <wire x1="14.5" y1="16.83" x2="12.7" y2="18.63" width="0.4064" layer="1"/>
-<contactref element="F1" pad="P$4"/>
-<contactref element="F1" pad="P$3"/>
-<wire x1="23.241" y1="7.1247" x2="23.241" y2="13.1953" width="0.4064" layer="1"/>
-<wire x1="23.241" y1="13.1953" x2="13.7287" y2="13.1953" width="0.4064" layer="1"/>
 <wire x1="13.7287" y1="13.1953" x2="10.922" y2="16.002" width="0.4064" layer="1"/>
 <wire x1="10.922" y1="16.002" x2="10.922" y2="18.034" width="0.4064" layer="1"/>
@@
 <wire x1="11.43" y1="18.542" x2="12.612" y2="18.542" width="0.4064" layer="1"/>
 <wire x1="12.612" y1="18.542" x2="12.7" y2="18.63" width="0.4064" layer="1"/>
+<contactref element="D1" pad="C"/>
+<wire x1="-3.81" y1="-9.283" x2="13.7287" y2="13.1953" width="0" layer="19" extent="1-1"/>
 </signal>
 <signal name="3.3V">
-<contactref element="C2" pad="1"/>
-<contactref element="U1" pad="5"/>
 <contactref element="TEENSY1" pad="1"/>
 <contactref element="AMPBRD" pad="3.3V"/>
-<wire x1="19.0801" y1="18.73" x2="21.49" y2="18.73" width="0.4064" layer="1"/>
-<wire x1="21.49" y1="18.73" x2="21.59" y2="18.63" width="0.4064" layer="1"/>
 <wire x1="3.81" y1="41.91" x2="3.81" y2="30.48" width="0.4064" layer="1"/>
 <wire x1="3.81" y1="30.48" x2="1.27" y2="27.94" width="0.4064" layer="1"/>
@@
 <wire x1="1.27" y1="21.59" x2="2.54" y2="20.32" width="0.4064" layer="1"/>
 <wire x1="20.32" y1="20.32" x2="21.59" y2="19.05" width="0.4064" layer="1"/>
-<wire x1="21.59" y1="19.05" x2="21.59" y2="18.63" width="0.4064" layer="1"/>
 <wire x1="3.81" y1="41.91" x2="3.81" y2="43.18" width="0.4064" layer="16"/>
 <wire x1="3.81" y1="43.18" x2="5.08" y2="44.45" width="0.4064" layer="16"/>
@@
 <wire x1="2.54" y1="20.32" x2="20.32" y2="20.32" width="0.4064" layer="1"/>
 <wire x1="42.7485" y1="17.78" x2="43.18" y2="17.78" width="0.4064" layer="1"/>
-<wire x1="21.59" y1="18.63" x2="23.28" y2="18.63" width="0.4064" layer="1"/>
 <wire x1="23.28" y1="18.63" x2="24.13" y2="17.78" width="0.4064" layer="1"/>
 <via x="24.13" y="17.78" extent="1-16" drill="0.6"/>
@@
 <wire x1="40.64" y1="19.05" x2="42.7485" y2="19.05" width="0.4064" layer="1"/>
 <wire x1="42.7485" y1="19.05" x2="42.7485" y2="17.78" width="0.4064" layer="1"/>
+<contactref element="D2" pad="C"/>
+<wire x1="21.59" y1="19.05" x2="23.28" y2="18.63" width="0" layer="19" extent="1-1"/>
+<wire x1="-3.81" y1="-13.093" x2="2.54" y2="20.32" width="0" layer="19" extent="1-1"/>
 </signal>
 <signal name="RO">
@@
 <wire x1="4.376" y1="18.796" x2="4.36" y2="18.78" width="0.4064" layer="1"/>
 </signal>
+<signal name="N$2">
+<contactref element="D5" pad="A"/>
+<contactref element="TEENSY2" pad="7"/>
+<wire x1="-3.81" y1="-26.277" x2="19.05" y2="26.67" width="0" layer="19" extent="1-1"/>
+</signal>
+<signal name="N$3">
+<contactref element="D4" pad="A"/>
+<contactref element="TEENSY2" pad="9"/>
+<wire x1="-3.81" y1="-22.467" x2="24.13" y2="26.67" width="0" layer="19" extent="1-1"/>
+</signal>
+<signal name="N$4">
+<contactref element="D3" pad="A"/>
+<contactref element="TEENSY2" pad="11"/>
+<wire x1="-3.81" y1="-18.657" x2="29.21" y2="26.67" width="0" layer="19" extent="1-1"/>
+</signal>
+<signal name="N$5">
+<contactref element="D1" pad="A"/>
+<contactref element="F1" pad="P$4"/>
+<contactref element="F1" pad="P$3"/>
+<wire x1="23.241" y1="7.1247" x2="23.241" y2="13.1953" width="0" layer="19" extent="1-1"/>
+<wire x1="-3.81" y1="-11.037" x2="23.241" y2="7.1247" width="0" layer="19" extent="1-1"/>
+</signal>
+<signal name="N$6">
+<contactref element="C2" pad="1"/>
+<contactref element="U1" pad="5"/>
+<wire x1="19.0801" y1="18.73" x2="21.49" y2="18.73" width="0.4064" layer="1"/>
+<wire x1="21.49" y1="18.73" x2="21.59" y2="18.63" width="0.4064" layer="1"/>
+<contactref element="D2" pad="A"/>
+<wire x1="-3.81" y1="-14.847" x2="19.0801" y2="18.73" width="0" layer="19" extent="1-1"/>
+</signal>
 </signals>

Commit message: Placed LEDs onto board.
Parts:
- moved D3 63.1 mm to (44.5, 22.9), turned to 270 degrees
- moved D4 62.9 mm to (40.6, 22.9), turned to 270 degrees
- moved D5 62.3 mm to (35.6, 22.9), turned to 270 degrees
- moved D2 37.8 mm to (8.89, 21.6)
- moved D1 22.9 mm to (3.81, 11.4), turned to 180 degrees
Connections:
- removed net N$5: D1.A, F1.P$3, F1.P$4
- removed net N$6: C2.1, D2.A, U1.5
- net 3.3V: now also C2.1, D2.A, U1.5; no longer D2.C
- net GND: now also D1.C, D2.C
- net N$2: now also D3.A, TEENSY2.14; no longer D5.A, TEENSY2.7
- net N$3: now also TEENSY2.13; no longer TEENSY2.9
- net N$4: now also D5.A, TEENSY2.12; no longer D3.A, TEENSY2.11
- net VCC: now also D1.A, F1.P$3, F1.P$4; no longer D1.C
Routing:
- net VCC: track 16.6 -> 52.7 mm, vias 0 -> 2
- net N$2: track 0.00 -> 8.83 mm
- net N$3: track 0.00 -> 7.05 mm
- net N$4: track 0.00 -> 5.02 mm
- net 3.3V: track 102.0 -> 107.0 mm
- net N$6: track 2.55 -> 0.00 mm
Changed lines of the file:
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@@
 <element name="U$1" library="BackplaneParts" package="MAX3491" value="MAX3491" x="36.83" y="11.43"/>
 <element name="F1" library="MotherboardParts" package="KEYSTONE_FUSE_3587" value="2A" x="16.51" y="10.16"/>
-<element name="D1" library="SparkFun-LED" package="LED-0603" value="" x="-3.81" y="-10.16"/>
-<element name="D2" library="SparkFun-LED" package="LED-0603" value="" x="-3.81" y="-13.97"/>
-<element name="D3" library="SparkFun-LED" package="LED-0603" value="" x="-3.81" y="-17.78"/>
-<element name="D4" library="SparkFun-LED" package="LED-0603" value="" x="-3.81" y="-21.59"/>
-<element name="D5" library="SparkFun-LED" package="LED-0603" value="" x="-3.81" y="-25.4"/>
+<element name="D1" library="SparkFun-LED" package="LED-0603" value="" x="3.81" y="11.43" rot="R180"/>
+<element name="D2" library="SparkFun-LED" package="LED-0603" value="" x="8.89" y="21.59"/>
+<element name="D3" library="SparkFun-LED" package="LED-0603" value="" x="44.45" y="22.86" rot="R270"/>
+<element name="D4" library="SparkFun-LED" package="LED-0603" value="" x="40.64" y="22.86" rot="R270"/>
+<element name="D5" library="SparkFun-LED" package="LED-0603" value="" x="35.56" y="22.86" rot="R270"/>
 </elements>
 <signals>
@@
 <contactref element="D4" pad="C"/>
 <contactref element="D3" pad="C"/>
-<wire x1="27.94" y1="50.8" x2="39.37" y2="41.91" width="0" layer="19" extent="1-1"/>
-<wire x1="25.4" y1="50.8" x2="27.94" y2="50.8" width="0" layer="19" extent="1-1"/>
-<wire x1="6.35" y1="41.91" x2="25.4" y2="50.8" width="0" layer="19" extent="1-1"/>
-<wire x1="3.81" y1="26.67" x2="6.35" y2="41.91" width="0" layer="19" extent="1-1"/>
-<wire x1="4.36" y1="16.78" x2="3.81" y2="26.67" width="0" layer="19" extent="1-1"/>
-<wire x1="12.7" y1="16.93" x2="4.36" y2="16.78" width="0" layer="19" extent="1-1"/>
-<wire x1="16.4799" y1="17.78" x2="12.7" y2="16.93" width="0" layer="19" extent="1-1"/>
-<wire x1="21.59" y1="16.93" x2="16.4799" y2="17.78" width="0" layer="19" extent="1-1"/>
-<wire x1="36.83" y1="12.7" x2="21.59" y2="16.93" width="0" layer="19" extent="1-1"/>
-<wire x1="36.83" y1="11.43" x2="36.83" y2="12.7" width="0" layer="19" extent="1-1"/>
-<wire x1="41.91" y1="2.54" x2="36.83" y2="11.43" width="0" layer="19" extent="1-1"/>
-<wire x1="-3.81" y1="-16.903" x2="4.36" y2="16.78" width="0" layer="19" extent="1-1"/>
-<wire x1="-3.81" y1="-20.713" x2="-3.81" y2="-16.903" width="0" layer="19" extent="1-1"/>
-<wire x1="-3.81" y1="-24.523" x2="-3.81" y2="-20.713" width="0" layer="19" extent="1-1"/>
+<contactref element="D2" pad="C"/>
+<contactref element="D1" pad="C"/>
 </signal>
 <signal name="VCC">
@@
 <wire x1="16.4799" y1="16.83" x2="14.5" y2="16.83" width="0.4064" layer="1"/>
 <wire x1="14.5" y1="16.83" x2="12.7" y2="18.63" width="0.4064" layer="1"/>
-<wire x1="13.7287" y1="13.1953" x2="10.922" y2="16.002" width="0.4064" layer="1"/>
-<wire x1="10.922" y1="16.002" x2="10.922" y2="18.034" width="0.4064" layer="1"/>
-<wire x1="10.922" y1="18.034" x2="11.43" y2="18.542" width="0.4064" layer="1"/>
-<wire x1="11.43" y1="18.542" x2="12.612" y2="18.542" width="0.4064" layer="1"/>
 <wire x1="12.612" y1="18.542" x2="12.7" y2="18.63" width="0.4064" layer="1"/>
-<contactref element="D1" pad="C"/>
-<wire x1="-3.81" y1="-9.283" x2="13.7287" y2="13.1953" width="0" layer="19" extent="1-1"/>
+<contactref element="F1" pad="P$4"/>
+<contactref element="F1" pad="P$3"/>
+<contactref element="D1" pad="A"/>
+<wire x1="23.241" y1="7.1247" x2="23.241" y2="11.811" width="0.4064" layer="1"/>
+<wire x1="23.241" y1="12.7" x2="23.241" y2="13.1953" width="0.4064" layer="1"/>
+<wire x1="12.612" y1="18.542" x2="12.192" y2="18.542" width="0.4064" layer="1"/>
+<wire x1="12.192" y1="18.542" x2="11.43" y2="17.78" width="0.4064" layer="1"/>
+<wire x1="11.43" y1="17.78" x2="11.43" y2="15.24" width="0.4064" layer="1"/>
+<wire x1="11.43" y1="15.24" x2="12.7" y2="13.97" width="0.4064" layer="1"/>
+<wire x1="12.7" y1="13.97" x2="22.86" y2="13.97" width="0.4064" layer="1"/>
+<wire x1="22.86" y1="13.97" x2="23.241" y2="13.589" width="0.4064" layer="1"/>
+<wire x1="23.241" y1="13.589" x2="23.241" y2="13.1953" width="0.4064" layer="1"/>
+<wire x1="3.81" y1="12.307" x2="4.687" y2="11.43" width="0.4064" layer="1"/>
+<wire x1="4.687" y1="11.43" x2="6.35" y2="11.43" width="0.4064" layer="1"/>
+<via x="6.35" y="11.43" extent="1-16" drill="0.6"/>
+<wire x1="6.35" y1="11.43" x2="7.62" y2="10.16" width="0.4064" layer="16"/>
+<wire x1="7.62" y1="10.16" x2="21.59" y2="10.16" width="0.4064" layer="16"/>
+<via x="21.59" y="10.16" extent="1-16" drill="0.6"/>
+<wire x1="21.59" y1="10.16" x2="23.241" y2="11.811" width="0.4064" layer="1"/>
+<wire x1="23.241" y1="11.811" x2="23.241" y2="12.7" width="0.4064" layer="1"/>
 </signal>
 <signal name="3.3V">
@@
 <wire x1="1.27" y1="27.94" x2="1.27" y2="21.59" width="0.4064" layer="1"/>
 <wire x1="1.27" y1="21.59" x2="2.54" y2="20.32" width="0.4064" layer="1"/>
-<wire x1="20.32" y1="20.32" x2="21.59" y2="19.05" width="0.4064" layer="1"/>
 <wire x1="3.81" y1="41.91" x2="3.81" y2="43.18" width="0.4064" layer="16"/>
 <wire x1="3.81" y1="43.18" x2="5.08" y2="44.45" width="0.4064" layer="16"/>
@@
 <contactref element="U$1" pad="VCC13"/>
 <contactref element="U$1" pad="VCC14"/>
-<wire x1="2.54" y1="20.32" x2="20.32" y2="20.32" width="0.4064" layer="1"/>
 <wire x1="42.7485" y1="17.78" x2="43.18" y2="17.78" width="0.4064" layer="1"/>
 <wire x1="23.28" y1="18.63" x2="24.13" y2="17.78" width="0.4064" layer="1"/>
@@
 <wire x1="40.64" y1="19.05" x2="42.7485" y2="19.05" width="0.4064" layer="1"/>
 <wire x1="42.7485" y1="19.05" x2="42.7485" y2="17.78" width="0.4064" layer="1"/>
-<contactref element="D2" pad="C"/>
-<wire x1="21.59" y1="19.05" x2="23.28" y2="18.63" width="0" layer="19" extent="1-1"/>
-<wire x1="-3.81" y1="-13.093" x2="2.54" y2="20.32" width="0" layer="19" extent="1-1"/>
+<contactref element="C2" pad="1"/>
+<contactref element="U1" pad="5"/>
+<wire x1="19.0801" y1="18.73" x2="21.49" y2="18.73" width="0.4064" layer="1"/>
+<wire x1="21.49" y1="18.73" x2="21.59" y2="18.63" width="0.4064" layer="1"/>
+<contactref element="D2" pad="A"/>
+<wire x1="2.54" y1="20.32" x2="8.497" y2="20.32" width="0.4064" layer="1"/>
+<wire x1="8.497" y1="20.32" x2="8.89" y2="20.713" width="0.4064" layer="1"/>
+<wire x1="21.59" y1="18.63" x2="21.59" y2="19.05" width="0.4064" layer="1"/>
+<wire x1="21.59" y1="19.05" x2="20.32" y2="20.32" width="0.4064" layer="1"/>
+<wire x1="20.32" y1="20.32" x2="9.283" y2="20.32" width="0.4064" layer="1"/>
+<wire x1="9.283" y1="20.32" x2="8.89" y2="20.713" width="0.4064" layer="1"/>
+<wire x1="23.28" y1="18.63" x2="21.59" y2="18.63" width="0.4064" layer="1"/>
 </signal>
 <signal name="RO">
@@
 </signal>
 <signal name="N$2">
-<contactref element="D5" pad="A"/>
-<contactref element="TEENSY2" pad="7"/>
-<wire x1="-3.81" y1="-26.277" x2="19.05" y2="26.67" width="0" layer="19" extent="1-1"/>
+<contactref element="D3" pad="A"/>
+<contactref element="TEENSY2" pad="14"/>
+<wire x1="43.573" y1="22.86" x2="43.573" y2="23.737" width="0.3048" layer="1"/>
+<wire x1="43.573" y1="23.737" x2="43.18" y2="24.13" width="0.3048" layer="1"/>
+<wire x1="43.18" y1="24.13" x2="39.37" y2="24.13" width="0.3048" layer="1"/>
+<wire x1="39.37" y1="24.13" x2="36.83" y2="26.67" width="0.3048" layer="1"/>
 </signal>
 <signal name="N$3">
 <contactref element="D4" pad="A"/>
-<contactref element="TEENSY2" pad="9"/>
-<wire x1="-3.81" y1="-22.467" x2="24.13" y2="26.67" width="0" layer="19" extent="1-1"/>
+<contactref element="TEENSY2" pad="13"/>
+<wire x1="39.763" y1="22.86" x2="39.37" y2="22.86" width="0.3048" layer="1"/>
+<wire x1="39.37" y1="22.86" x2="38.1" y2="24.13" width="0.3048" layer="1"/>
+<wire x1="38.1" y1="24.13" x2="36.83" y2="24.13" width="0.3048" layer="1"/>
+<wire x1="36.83" y1="24.13" x2="34.29" y2="26.67" width="0.3048" layer="1"/>
 </signal>
 <signal name="N$4">
-<contactref element="D3" pad="A"/>
-<contactref element="TEENSY2" pad="11"/>
-<wire x1="-3.81" y1="-18.657" x2="29.21" y2="26.67" width="0" layer="19" extent="1-1"/>
-</signal>
-<signal name="N$5">
-<contactref element="D1" pad="A"/>
-<contactref element="F1" pad="P$4"/>
-<contactref element="F1" pad="P$3"/>
-<wire x1="23.241" y1="7.1247" x2="23.241" y2="13.1953" width="0" layer="19" extent="1-1"/>
-<wire x1="-3.81" y1="-11.037" x2="23.241" y2="7.1247" width="0" layer="19" extent="1-1"/>
-</signal>
-<signal name="N$6">
-<contactref element="C2" pad="1"/>
-<contactref element="U1" pad="5"/>
-<wire x1="19.0801" y1="18.73" x2="21.49" y2="18.73" width="0.4064" layer="1"/>
-<wire x1="21.49" y1="18.73" x2="21.59" y2="18.63" width="0.4064" layer="1"/>
-<contactref element="D2" pad="A"/>
-<wire x1="-3.81" y1="-14.847" x2="19.0801" y2="18.73" width="0" layer="19" extent="1-1"/>
+<contactref element="D5" pad="A"/>
+<contactref element="TEENSY2" pad="12"/>
+<wire x1="34.683" y1="22.86" x2="34.683" y2="23.737" width="0.3048" layer="1"/>
+<wire x1="34.683" y1="23.737" x2="31.75" y2="26.67" width="0.3048" layer="1"/>
 </signal>
 </signals>
