File: TeensySonarBoard.brd (EAGLE design)
At the start: 59.7 x 53.3 mm, 16 parts, among them J5 RJ45, U1 MIC5219 3.3V

Commit message: fixed ledissues
Parts:
- added R1, R2, R3, R4, R5: (no value), resistor:R0603
- moved D2 26.6 mm to (33.0, 10.4), turned to 180 degrees
- moved D1 24.9 mm to (28.7, 10.2)
- moved D5 20.7 mm to (48.0, 39.4)
- moved D4 15.8 mm to (48.0, 36.8)
- moved D3 12.0 mm to (48.0, 34.3)
Connections:
- new net N$5: D1.C, R5.2
- new net N$6: D2.C, R4.2
- new net N$7: D3.C, R1.1
- new net N$8: D4.C, R2.1
- new net N$9: D5.C, R3.1
- net GND: now also R1.2, R2.2, R3.2, R4.1, R5.1; no longer D1.C, D2.C, D3.C, D4.C, D5.C
Routing:
- net N$4: track 5.02 -> 21.1 mm
- net VCC: track 52.7 -> 38.0 mm, vias 2 -> 0
- net 3.3V: track 107.0 -> 118.3 mm
- net N$3: track 7.05 -> 17.8 mm
- net N$2: track 8.83 -> 14.2 mm
- net N$9: track 0.00 -> 3.10 mm
- net N$8: track 0.00 -> 3.10 mm
- net N$7: track 0.00 -> 3.10 mm
- net N$5: track 0.00 -> 2.16 mm
- net N$6: track 0.00 -> 1.99 mm
Other:
- board size 59.7 x 53.3 mm -> 61 x 53.3 mm
- board text added: "+9V"
- board text added: "3.3V"
Changed lines of the file:
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@@
 <setting verticaltext="up"/>
 </settings>
-<grid distance="0.05" unitdist="inch" unit="inch" style="lines" multiple="1" display="yes" altdistance="0.025" altunitdist="inch" altunit="inch"/>
+<grid distance="0.01" unitdist="inch" unit="inch" style="lines" multiple="1" display="yes" altdistance="0.025" altunitdist="inch" altunit="inch"/>
 <layers>
 <layer number="1" name="Top" color="4" fill="1" visible="yes" active="yes"/>
@@
 <layer number="49" name="Reference" color="7" fill="1" visible="yes" active="yes"/>
 <layer number="50" name="dxf" color="7" fill="1" visible="no" active="no"/>
-<layer number="51" name="tDocu" color="7" fill="1" visible="yes" active="yes"/>
-<layer number="52" name="bDocu" color="7" fill="1" visible="yes" active="yes"/>
+<layer number="51" name="tDocu" color="7" fill="1" visible="no" active="yes"/>
+<layer number="52" name="bDocu" color="7" fill="1" visible="no" active="yes"/>
 <layer number="53" name="tGND_GNDA" color="7" fill="9" visible="no" active="no"/>
 <layer number="54" name="bGND_GNDA" color="1" fill="9" visible="no" active="no"/>
@@
 <board>
 <plain>
-<wire x1="0" y1="0" x2="59.69" y2="0" width="0" layer="20"/>
-<wire x1="59.69" y1="0" x2="59.69" y2="53.34" width="0" layer="20"/>
-<wire x1="59.69" y1="53.34" x2="0" y2="53.34" width="0" layer="20"/>
+<wire x1="0" y1="0" x2="60.96" y2="0" width="0" layer="20"/>
+<wire x1="60.96" y1="0" x2="60.96" y2="53.34" width="0" layer="20"/>
+<wire x1="60.96" y1="53.34" x2="0" y2="53.34" width="0" layer="20"/>
 <wire x1="0" y1="53.34" x2="0" y2="0" width="0" layer="20"/>
+<text x="31.242" y="12.192" size="1.4224" layer="21">3.3V</text>
+<text x="26.67" y="12.192" size="1.4224" layer="21">+9V</text>
 </plain>
 <attributes>
@@
 </class>
 </classes>
-<designrules name="GoldPhoenix">
+<designrules name="GoldPhoenix *">
 <description language="en">
 &lt;b&gt;Gold Phoenix PCB Design Rules&lt;/b&gt;
@@
 <param name="mdViaViaSameLayer" value="8mil"/>
 <param name="mnLayersViaInSmd" value="2"/>
-<param name="mdCopperDimension" value="10mil"/>
+<param name="mdCopperDimension" value="20mil"/>
 <param name="mdDrill" value="8mil"/>
 <param name="mdSmdStop" value="0mil"/>
@@
 <element name="U$1" library="BackplaneParts" package="MAX3491" value="MAX3491" x="36.83" y="11.43"/>
 <element name="F1" library="MotherboardParts" package="KEYSTONE_FUSE_3587" value="2A" x="16.51" y="10.16"/>
-<element name="D1" library="SparkFun-LED" package="LED-0603" value="" x="3.81" y="11.43" rot="R180"/>
-<element name="D2" library="SparkFun-LED" package="LED-0603" value="" x="8.89" y="21.59"/>
-<element name="D3" library="SparkFun-LED" package="LED-0603" value="" x="44.45" y="22.86" rot="R270"/>
-<element name="D4" library="SparkFun-LED" package="LED-0603" value="" x="40.64" y="22.86" rot="R270"/>
-<element name="D5" library="SparkFun-LED" package="LED-0603" value="" x="35.56" y="22.86" rot="R270"/>
+<element name="D1" library="SparkFun-LED" package="LED-0603" value="" x="28.702" y="10.16" rot="R180"/>
+<element name="D2" library="SparkFun-LED" package="LED-0603" value="" x="33.02" y="10.414" rot="R180"/>
+<element name="D3" library="SparkFun-LED" package="LED-0603" value="" x="48.006" y="34.29" rot="R270"/>
+<element name="D4" library="SparkFun-LED" package="LED-0603" value="" x="48.006" y="36.83" rot="R270"/>
+<element name="D5" library="SparkFun-LED" package="LED-0603" value="" x="48.006" y="39.37" rot="R270"/>
+<element name="R1" library="resistor" package="R0603" value="" x="52.832" y="34.29"/>
+<element name="R2" library="resistor" package="R0603" value="" x="52.832" y="36.83"/>
+<element name="R3" library="resistor" package="R0603" value="" x="52.832" y="39.37"/>
+<element name="R4" library="resistor" package="R0603" value="" x="34.036" y="7.62" rot="R180"/>
+<element name="R5" library="resistor" package="R0603" value="" x="28.956" y="7.366" rot="R180"/>
 </elements>
 <signals>
@@
 <vertex x="59.69" y="0"/>
 </polygon>
-<contactref element="D5" pad="C"/>
-<contactref element="D4" pad="C"/>
-<contactref element="D3" pad="C"/>
-<contactref element="D2" pad="C"/>
-<contactref element="D1" pad="C"/>
+<contactref element="R5" pad="1"/>
+<contactref element="R4" pad="1"/>
+<contactref element="R1" pad="2"/>
+<contactref element="R2" pad="2"/>
+<contactref element="R3" pad="2"/>
 </signal>
 <signal name="VCC">
@@
 <contactref element="F1" pad="P$3"/>
 <contactref element="D1" pad="A"/>
-<wire x1="23.241" y1="7.1247" x2="23.241" y2="11.811" width="0.4064" layer="1"/>
-<wire x1="23.241" y1="12.7" x2="23.241" y2="13.1953" width="0.4064" layer="1"/>
+<wire x1="23.241" y1="7.1247" x2="23.241" y2="13.1953" width="0.4064" layer="1"/>
 <wire x1="12.612" y1="18.542" x2="12.192" y2="18.542" width="0.4064" layer="1"/>
 <wire x1="12.192" y1="18.542" x2="11.43" y2="17.78" width="0.4064" layer="1"/>
@@
 <wire x1="22.86" y1="13.97" x2="23.241" y2="13.589" width="0.4064" layer="1"/>
 <wire x1="23.241" y1="13.589" x2="23.241" y2="13.1953" width="0.4064" layer="1"/>
-<wire x1="3.81" y1="12.307" x2="4.687" y2="11.43" width="0.4064" layer="1"/>
-<wire x1="4.687" y1="11.43" x2="6.35" y2="11.43" width="0.4064" layer="1"/>
-<via x="6.35" y="11.43" extent="1-16" drill="0.6"/>
-<wire x1="6.35" y1="11.43" x2="7.62" y2="10.16" width="0.4064" layer="16"/>
-<wire x1="7.62" y1="10.16" x2="21.59" y2="10.16" width="0.4064" layer="16"/>
-<via x="21.59" y="10.16" extent="1-16" drill="0.6"/>
-<wire x1="21.59" y1="10.16" x2="23.241" y2="11.811" width="0.4064" layer="1"/>
-<wire x1="23.241" y1="11.811" x2="23.241" y2="12.7" width="0.4064" layer="1"/>
+<wire x1="23.241" y1="13.1953" x2="26.5437" y2="13.1953" width="0.4064" layer="1"/>
+<wire x1="26.5437" y1="13.1953" x2="28.702" y2="11.037" width="0.4064" layer="1"/>
 </signal>
 <signal name="3.3V">
@@
 <wire x1="21.49" y1="18.73" x2="21.59" y2="18.63" width="0.4064" layer="1"/>
 <contactref element="D2" pad="A"/>
-<wire x1="2.54" y1="20.32" x2="8.497" y2="20.32" width="0.4064" layer="1"/>
-<wire x1="8.497" y1="20.32" x2="8.89" y2="20.713" width="0.4064" layer="1"/>
 <wire x1="21.59" y1="18.63" x2="21.59" y2="19.05" width="0.4064" layer="1"/>
 <wire x1="21.59" y1="19.05" x2="20.32" y2="20.32" width="0.4064" layer="1"/>
-<wire x1="20.32" y1="20.32" x2="9.283" y2="20.32" width="0.4064" layer="1"/>
-<wire x1="9.283" y1="20.32" x2="8.89" y2="20.713" width="0.4064" layer="1"/>
+<wire x1="20.32" y1="20.32" x2="2.54" y2="20.32" width="0.4064" layer="1"/>
 <wire x1="23.28" y1="18.63" x2="21.59" y2="18.63" width="0.4064" layer="1"/>
+<wire x1="33.02" y1="11.291" x2="31.127" y2="11.291" width="0.4064" layer="1"/>
+<wire x1="31.127" y1="11.291" x2="29.718" y2="12.7" width="0.4064" layer="1"/>
+<wire x1="29.718" y1="12.7" x2="29.21" y2="12.7" width="0.4064" layer="1"/>
+<wire x1="29.21" y1="12.7" x2="24.13" y2="17.78" width="0.4064" layer="1"/>
 </signal>
 <signal name="RO">
@@
 <contactref element="D3" pad="A"/>
 <contactref element="TEENSY2" pad="14"/>
-<wire x1="43.573" y1="22.86" x2="43.573" y2="23.737" width="0.3048" layer="1"/>
-<wire x1="43.573" y1="23.737" x2="43.18" y2="24.13" width="0.3048" layer="1"/>
-<wire x1="43.18" y1="24.13" x2="39.37" y2="24.13" width="0.3048" layer="1"/>
-<wire x1="39.37" y1="24.13" x2="36.83" y2="26.67" width="0.3048" layer="1"/>
+<wire x1="36.83" y1="26.67" x2="36.83" y2="27.94" width="0.4064" layer="1"/>
+<wire x1="36.83" y1="27.94" x2="43.18" y2="34.29" width="0.4064" layer="1"/>
+<wire x1="43.18" y1="34.29" x2="47.129" y2="34.29" width="0.4064" layer="1"/>
 </signal>
 <signal name="N$3">
 <contactref element="D4" pad="A"/>
 <contactref element="TEENSY2" pad="13"/>
-<wire x1="39.763" y1="22.86" x2="39.37" y2="22.86" width="0.3048" layer="1"/>
-<wire x1="39.37" y1="22.86" x2="38.1" y2="24.13" width="0.3048" layer="1"/>
-<wire x1="38.1" y1="24.13" x2="36.83" y2="24.13" width="0.3048" layer="1"/>
-<wire x1="36.83" y1="24.13" x2="34.29" y2="26.67" width="0.3048" layer="1"/>
+<wire x1="34.29" y1="26.67" x2="34.29" y2="27.94" width="0.4064" layer="1"/>
+<wire x1="34.29" y1="27.94" x2="43.18" y2="36.83" width="0.4064" layer="1"/>
+<wire x1="43.18" y1="36.83" x2="47.129" y2="36.83" width="0.4064" layer="1"/>
 </signal>
 <signal name="N$4">
 <contactref element="D5" pad="A"/>
 <contactref element="TEENSY2" pad="12"/>
-<wire x1="34.683" y1="22.86" x2="34.683" y2="23.737" width="0.3048" layer="1"/>
-<wire x1="34.683" y1="23.737" x2="31.75" y2="26.67" width="0.3048" layer="1"/>
+<wire x1="31.75" y1="26.67" x2="31.75" y2="27.432" width="0.4064" layer="1"/>
+<wire x1="31.75" y1="27.432" x2="43.688" y2="39.37" width="0.4064" layer="1"/>
+<wire x1="43.688" y1="39.37" x2="47.129" y2="39.37" width="0.4064" layer="1"/>
+</signal>
+<signal name="N$5">
+<contactref element="R5" pad="2"/>
+<contactref element="D1" pad="C"/>
+<wire x1="28.702" y1="9.283" x2="28.702" y2="7.962" width="0.4064" layer="1"/>
+<wire x1="28.702" y1="7.962" x2="28.106" y2="7.366" width="0.4064" layer="1"/>
+</signal>
+<signal name="N$6">
+<contactref element="R4" pad="2"/>
+<contactref element="D2" pad="C"/>
+<wire x1="33.02" y1="9.537" x2="33.02" y2="7.786" width="0.4064" layer="1"/>
+<wire x1="33.02" y1="7.786" x2="33.186" y2="7.62" width="0.4064" layer="1"/>
+</signal>
+<signal name="N$7">
+<contactref element="D3" pad="C"/>
+<contactref element="R1" pad="1"/>
+<wire x1="48.883" y1="34.29" x2="51.982" y2="34.29" width="0.4064" layer="1"/>
+</signal>
+<signal name="N$8">
+<contactref element="D4" pad="C"/>
+<contactref element="R2" pad="1"/>
+<wire x1="48.883" y1="36.83" x2="51.982" y2="36.83" width="0.4064" layer="1"/>
+</signal>
+<signal name="N$9">
+<contactref element="D5" pad="C"/>
+<contactref element="R3" pad="1"/>
+<wire x1="48.883" y1="39.37" x2="51.982" y2="39.37" width="0.4064" layer="1"/>
 </signal>
 </signals>
