File: TeensySonarBoard.sch (EAGLE design)
At the start: 10 parts, among them J5 RJ45, U1 MIC5219 3.3V

Commit message: Added a 2A fuse to the board to meet MATE requirements.
Parts:
- added F1: 2A, MotherboardParts:KEYSTONE_FUSE_3587
Connections:
- new net N$1: BATT.2, F1.P$1
- net VCC: now also F1.P$2; no longer BATT.2
Changed lines of the file:
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@@
 <part name="GND10" library="SparkFun-Aesthetics" deviceset="GND" device=""/>
 <part name="SUPPLY7" library="SparkFun-Aesthetics" deviceset="3.3V" device=""/>
+<part name="F1" library="MotherboardParts" deviceset="KEYSTONE_FUSE_3587" device="" value="2A"/>
 </parts>
 <sheets>
@@
 <instance part="GND6" gate="1" x="109.22" y="132.08"/>
 <instance part="AMPBRD" gate="G$1" x="58.42" y="121.92"/>
-<instance part="SUPPLY1" gate="G$1" x="15.24" y="68.58"/>
+<instance part="SUPPLY1" gate="G$1" x="17.78" y="73.66"/>
 <instance part="GND1" gate="1" x="15.24" y="38.1"/>
 <instance part="GND3" gate="1" x="40.64" y="93.98"/>
@@
 <instance part="GND10" gate="1" x="162.56" y="43.18"/>
 <instance part="SUPPLY7" gate="G$1" x="198.12" y="76.2"/>
+<instance part="F1" gate="G$1" x="17.78" y="63.5" rot="R90"/>
 </instances>
 <busses>
@@
 </segment>
 <segment>
+<pinref part="F1" gate="G$1" pin="P$2"/>
 <pinref part="SUPPLY1" gate="G$1" pin="VCC"/>
-<pinref part="BATT" gate="G$1" pin="2"/>
-<wire x1="15.24" y1="68.58" x2="15.24" y2="55.88" width="0.1524" layer="91"/>
+<wire x1="17.78" y1="68.58" x2="17.78" y2="73.66" width="0.1524" layer="91"/>
 </segment>
 </net>
@@
 </segment>
 </net>
+<net name="N$1" class="0">
+<segment>
+<pinref part="BATT" gate="G$1" pin="2"/>
+<pinref part="F1" gate="G$1" pin="P$1"/>
+<wire x1="15.24" y1="55.88" x2="17.78" y2="55.88" width="0.1524" layer="91"/>
+<wire x1="17.78" y1="55.88" x2="17.78" y2="58.42" width="0.1524" layer="91"/>
+</segment>
+</net>
