File: TeensySonarBoard.sch (EAGLE design)
At the start: 11 parts, among them J5 RJ45, U1 MIC5219 3.3V

Commit message: Initial placement of diagnostic LEDs.
Parts:
- added D1, D2, D3, D4, D5: (no value), SparkFun-LED:LED0603
Connections:
- new net N$2: D5.A, TEENSY2.7
- new net N$3: D4.A, TEENSY2.9
- new net N$4: D3.A, TEENSY2.11
- new net N$5: D1.A, F1.P$2
- new net N$6: C2.1, D2.A, U1.OUT
- net 3.3V: now also D2.C; no longer C2.1, U1.OUT
- net GND: now also D3.C, D4.C, D5.C
- net VCC: now also D1.C; no longer F1.P$2
Changed lines of the file:
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@@
 <part name="SUPPLY7" library="SparkFun-Aesthetics" deviceset="3.3V" device=""/>
 <part name="F1" library="MotherboardParts" deviceset="KEYSTONE_FUSE_3587" device="" value="2A"/>
+<part name="D1" library="SparkFun-LED" deviceset="LED" device="0603"/>
+<part name="D2" library="SparkFun-LED" deviceset="LED" device="0603"/>
+<part name="D3" library="SparkFun-LED" deviceset="LED" device="0603"/>
+<part name="D4" library="SparkFun-LED" deviceset="LED" device="0603"/>
+<part name="D5" library="SparkFun-LED" deviceset="LED" device="0603"/>
+<part name="GND9" library="SparkFun-Aesthetics" deviceset="GND" device=""/>
 </parts>
 <sheets>
@@
 </plain>
 <instances>
-<instance part="SUPPLY4" gate="G$1" x="68.58" y="55.88"/>
+<instance part="SUPPLY4" gate="G$1" x="68.58" y="66.04"/>
 <instance part="GND4" gate="1" x="40.64" y="38.1"/>
 <instance part="SUPPLY2" gate="G$1" x="33.02" y="55.88"/>
@@
 <instance part="GND6" gate="1" x="109.22" y="132.08"/>
 <instance part="AMPBRD" gate="G$1" x="58.42" y="121.92"/>
-<instance part="SUPPLY1" gate="G$1" x="17.78" y="73.66"/>
+<instance part="SUPPLY1" gate="G$1" x="17.78" y="83.82"/>
 <instance part="GND1" gate="1" x="15.24" y="38.1"/>
 <instance part="GND3" gate="1" x="40.64" y="93.98"/>
@@
 <instance part="SUPPLY7" gate="G$1" x="198.12" y="76.2"/>
 <instance part="F1" gate="G$1" x="17.78" y="63.5" rot="R90"/>
+<instance part="D1" gate="G$1" x="17.78" y="73.66" rot="R180"/>
+<instance part="D2" gate="G$1" x="68.58" y="58.42" rot="R180"/>
+<instance part="D3" gate="G$1" x="170.18" y="134.62" rot="R90"/>
+<instance part="D4" gate="G$1" x="170.18" y="127" rot="R90"/>
+<instance part="D5" gate="G$1" x="170.18" y="119.38" rot="R90"/>
+<instance part="GND9" gate="1" x="180.34" y="114.3"/>
 </instances>
 <busses>
@@
 <junction x="162.56" y="48.26"/>
 </segment>
+<segment>
+<pinref part="D5" gate="G$1" pin="C"/>
+<pinref part="GND9" gate="1" pin="GND"/>
+<wire x1="175.26" y1="119.38" x2="180.34" y2="119.38" width="0.1524" layer="91"/>
+<wire x1="180.34" y1="119.38" x2="180.34" y2="116.84" width="0.1524" layer="91"/>
+<pinref part="D4" gate="G$1" pin="C"/>
+<wire x1="175.26" y1="127" x2="180.34" y2="127" width="0.1524" layer="91"/>
+<wire x1="180.34" y1="127" x2="180.34" y2="119.38" width="0.1524" layer="91"/>
+<junction x="180.34" y="119.38"/>
+<pinref part="D3" gate="G$1" pin="C"/>
+<wire x1="175.26" y1="134.62" x2="180.34" y2="134.62" width="0.1524" layer="91"/>
+<wire x1="180.34" y1="134.62" x2="180.34" y2="127" width="0.1524" layer="91"/>
+<junction x="180.34" y="127"/>
+</segment>
 </net>
 <net name="VCC" class="0">
@@
 </segment>
 <segment>
-<pinref part="F1" gate="G$1" pin="P$2"/>
+<pinref part="D1" gate="G$1" pin="C"/>
 <pinref part="SUPPLY1" gate="G$1" pin="VCC"/>
-<wire x1="17.78" y1="68.58" x2="17.78" y2="73.66" width="0.1524" layer="91"/>
+<wire x1="17.78" y1="78.74" x2="17.78" y2="83.82" width="0.1524" layer="91"/>
 </segment>
 </net>
 <net name="3.3V" class="0">
-<segment>
-<pinref part="C2" gate="G$1" pin="1"/>
-<pinref part="SUPPLY4" gate="G$1" pin="3.3V"/>
-<wire x1="68.58" y1="50.8" x2="68.58" y2="53.34" width="0.1524" layer="91"/>
-<pinref part="U1" gate="G$1" pin="OUT"/>
-<wire x1="68.58" y1="53.34" x2="68.58" y2="55.88" width="0.1524" layer="91"/>
-<wire x1="60.96" y1="53.34" x2="68.58" y2="53.34" width="0.1524" layer="91"/>
-<junction x="68.58" y="53.34"/>
-</segment>
 <segment>
 <pinref part="TEENSY1" gate="G$1" pin="1"/>
@@
 <junction x="198.12" y="73.66"/>
 </segment>
+<segment>
+<pinref part="SUPPLY4" gate="G$1" pin="3.3V"/>
+<pinref part="D2" gate="G$1" pin="C"/>
+<wire x1="68.58" y1="66.04" x2="68.58" y2="63.5" width="0.1524" layer="91"/>
+</segment>
 </net>
 <net name="RO" class="0">
@@
 </segment>
 </net>
+<net name="N$2" class="0">
+<segment>
+<pinref part="D5" gate="G$1" pin="A"/>
+<wire x1="167.64" y1="119.38" x2="165.1" y2="119.38" width="0.1524" layer="91"/>
+<wire x1="165.1" y1="119.38" x2="165.1" y2="116.84" width="0.1524" layer="91"/>
+<pinref part="TEENSY2" gate="G$1" pin="7"/>
+<wire x1="165.1" y1="116.84" x2="160.02" y2="116.84" width="0.1524" layer="91"/>
+</segment>
+</net>
+<net name="N$3" class="0">
+<segment>
+<pinref part="D4" gate="G$1" pin="A"/>
+<wire x1="167.64" y1="127" x2="167.64" y2="121.92" width="0.1524" layer="91"/>
+<pinref part="TEENSY2" gate="G$1" pin="9"/>
+<wire x1="167.64" y1="121.92" x2="160.02" y2="121.92" width="0.1524" layer="91"/>
+</segment>
+</net>
+<net name="N$4" class="0">
+<segment>
+<pinref part="D3" gate="G$1" pin="A"/>
+<wire x1="167.64" y1="134.62" x2="165.1" y2="134.62" width="0.1524" layer="91"/>
+<wire x1="165.1" y1="134.62" x2="165.1" y2="127" width="0.1524" layer="91"/>
+<pinref part="TEENSY2" gate="G$1" pin="11"/>
+<wire x1="165.1" y1="127" x2="160.02" y2="127" width="0.1524" layer="91"/>
+</segment>
+</net>
+<net name="N$5" class="0">
+<segment>
+<pinref part="D1" gate="G$1" pin="A"/>
+<pinref part="F1" gate="G$1" pin="P$2"/>
+<wire x1="17.78" y1="71.12" x2="17.78" y2="68.58" width="0.1524" layer="91"/>
+</segment>
+</net>
+<net name="N$6" class="0">
+<segment>
+<pinref part="C2" gate="G$1" pin="1"/>
+<wire x1="68.58" y1="50.8" x2="68.58" y2="53.34" width="0.1524" layer="91"/>
+<pinref part="U1" gate="G$1" pin="OUT"/>
+<wire x1="60.96" y1="53.34" x2="68.58" y2="53.34" width="0.1524" layer="91"/>
+<pinref part="D2" gate="G$1" pin="A"/>
+<wire x1="68.58" y1="55.88" x2="68.58" y2="53.34" width="0.1524" layer="91"/>
+<junction x="68.58" y="53.34"/>
+</segment>
+</net>

Commit message: Placed LEDs onto board.
Connections:
- removed net N$5: D1.A, F1.P$2
- removed net N$6: C2.1, D2.A, U1.OUT
- net 3.3V: now also C2.1, D2.A, U1.OUT; no longer D2.C
- net GND: now also D1.C, D2.C
- net N$2: now also D3.A, TEENSY2.14; no longer D5.A, TEENSY2.7
- net N$3: now also TEENSY2.13; no longer TEENSY2.9
- net N$4: now also D5.A, TEENSY2.12; no longer D3.A, TEENSY2.11
- net VCC: now also D1.A, F1.P$2; no longer D1.C
Other:
- moved on the sheet: D1, D2
Changed lines of the file:
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@@
 </classes>
 <parts>
-<part name="SUPPLY4" library="SparkFun-Aesthetics" deviceset="3.3V" device=""/>
 <part name="GND4" library="SparkFun-Aesthetics" deviceset="GND" device=""/>
 <part name="SUPPLY2" library="SparkFun-Aesthetics" deviceset="VCC" device="" value="9V"/>
@@
 <part name="D5" library="SparkFun-LED" deviceset="LED" device="0603"/>
 <part name="GND9" library="SparkFun-Aesthetics" deviceset="GND" device=""/>
+<part name="SUPPLY4" library="SparkFun-Aesthetics" deviceset="3.3V" device=""/>
+<part name="GND11" library="SparkFun-Aesthetics" deviceset="GND" device=""/>
+<part name="SUPPLY6" library="SparkFun-Aesthetics" deviceset="3.3V" device=""/>
+<part name="SUPPLY8" library="SparkFun-Aesthetics" deviceset="VCC" device="" value="9V"/>
+<part name="GND12" library="SparkFun-Aesthetics" deviceset="GND" device=""/>
 </parts>
 <sheets>
@@
 </plain>
 <instances>
-<instance part="SUPPLY4" gate="G$1" x="68.58" y="66.04"/>
 <instance part="GND4" gate="1" x="40.64" y="38.1"/>
 <instance part="SUPPLY2" gate="G$1" x="33.02" y="55.88"/>
@@
 <instance part="GND6" gate="1" x="109.22" y="132.08"/>
 <instance part="AMPBRD" gate="G$1" x="58.42" y="121.92"/>
-<instance part="SUPPLY1" gate="G$1" x="17.78" y="83.82"/>
+<instance part="SUPPLY1" gate="G$1" x="17.78" y="71.12"/>
 <instance part="GND1" gate="1" x="15.24" y="38.1"/>
 <instance part="GND3" gate="1" x="40.64" y="93.98"/>
@@
 <instance part="SUPPLY7" gate="G$1" x="198.12" y="76.2"/>
 <instance part="F1" gate="G$1" x="17.78" y="63.5" rot="R90"/>
-<instance part="D1" gate="G$1" x="17.78" y="73.66" rot="R180"/>
-<instance part="D2" gate="G$1" x="68.58" y="58.42" rot="R180"/>
+<instance part="D1" gate="G$1" x="7.62" y="76.2"/>
+<instance part="D2" gate="G$1" x="83.82" y="58.42"/>
 <instance part="D3" gate="G$1" x="170.18" y="134.62" rot="R90"/>
 <instance part="D4" gate="G$1" x="170.18" y="127" rot="R90"/>
 <instance part="D5" gate="G$1" x="170.18" y="119.38" rot="R90"/>
 <instance part="GND9" gate="1" x="180.34" y="114.3"/>
+<instance part="SUPPLY4" gate="G$1" x="68.58" y="55.88"/>
+<instance part="GND11" gate="1" x="83.82" y="45.72"/>
+<instance part="SUPPLY6" gate="G$1" x="83.82" y="66.04"/>
+<instance part="SUPPLY8" gate="G$1" x="7.62" y="81.28"/>
+<instance part="GND12" gate="1" x="7.62" y="66.04"/>
 </instances>
 <busses>
@@
 <junction x="180.34" y="127"/>
 </segment>
+<segment>
+<pinref part="D2" gate="G$1" pin="C"/>
+<pinref part="GND11" gate="1" pin="GND"/>
+<wire x1="83.82" y1="53.34" x2="83.82" y2="48.26" width="0.1524" layer="91"/>
+</segment>
+<segment>
+<pinref part="D1" gate="G$1" pin="C"/>
+<pinref part="GND12" gate="1" pin="GND"/>
+<wire x1="7.62" y1="71.12" x2="7.62" y2="68.58" width="0.1524" layer="91"/>
+</segment>
 </net>
 <net name="VCC" class="0">
@@
 </segment>
 <segment>
-<pinref part="D1" gate="G$1" pin="C"/>
+<pinref part="F1" gate="G$1" pin="P$2"/>
 <pinref part="SUPPLY1" gate="G$1" pin="VCC"/>
-<wire x1="17.78" y1="78.74" x2="17.78" y2="83.82" width="0.1524" layer="91"/>
+<wire x1="17.78" y1="71.12" x2="17.78" y2="68.58" width="0.1524" layer="91"/>
+</segment>
+<segment>
+<pinref part="D1" gate="G$1" pin="A"/>
+<pinref part="SUPPLY8" gate="G$1" pin="VCC"/>
+<wire x1="7.62" y1="78.74" x2="7.62" y2="81.28" width="0.1524" layer="91"/>
 </segment>
 </net>
@@
 </segment>
 <segment>
+<pinref part="C2" gate="G$1" pin="1"/>
+<wire x1="68.58" y1="50.8" x2="68.58" y2="53.34" width="0.1524" layer="91"/>
+<pinref part="U1" gate="G$1" pin="OUT"/>
+<wire x1="60.96" y1="53.34" x2="68.58" y2="53.34" width="0.1524" layer="91"/>
 <pinref part="SUPPLY4" gate="G$1" pin="3.3V"/>
-<pinref part="D2" gate="G$1" pin="C"/>
-<wire x1="68.58" y1="66.04" x2="68.58" y2="63.5" width="0.1524" layer="91"/>
+<wire x1="68.58" y1="53.34" x2="68.58" y2="55.88" width="0.1524" layer="91"/>
+<junction x="68.58" y="53.34"/>
+</segment>
+<segment>
+<pinref part="SUPPLY6" gate="G$1" pin="3.3V"/>
+<pinref part="D2" gate="G$1" pin="A"/>
+<wire x1="83.82" y1="66.04" x2="83.82" y2="60.96" width="0.1524" layer="91"/>
 </segment>
 </net>
@@
 <net name="N$2" class="0">
 <segment>
+<pinref part="D3" gate="G$1" pin="A"/>
+<pinref part="TEENSY2" gate="G$1" pin="14"/>
+<wire x1="167.64" y1="134.62" x2="160.02" y2="134.62" width="0.1524" layer="91"/>
+</segment>
+</net>
+<net name="N$3" class="0">
+<segment>
+<pinref part="D4" gate="G$1" pin="A"/>
+<wire x1="167.64" y1="127" x2="167.64" y2="132.08" width="0.1524" layer="91"/>
+<pinref part="TEENSY2" gate="G$1" pin="13"/>
+<wire x1="167.64" y1="132.08" x2="160.02" y2="132.08" width="0.1524" layer="91"/>
+</segment>
+</net>
+<net name="N$4" class="0">
+<segment>
 <pinref part="D5" gate="G$1" pin="A"/>
 <wire x1="167.64" y1="119.38" x2="165.1" y2="119.38" width="0.1524" layer="91"/>
-<wire x1="165.1" y1="119.38" x2="165.1" y2="116.84" width="0.1524" layer="91"/>
-<pinref part="TEENSY2" gate="G$1" pin="7"/>
-<wire x1="165.1" y1="116.84" x2="160.02" y2="116.84" width="0.1524" layer="91"/>
-</segment>
-</net>
-<net name="N$3" class="0">
-<segment>
-<pinref part="D4" gate="G$1" pin="A"/>
-<wire x1="167.64" y1="127" x2="167.64" y2="121.92" width="0.1524" layer="91"/>
-<pinref part="TEENSY2" gate="G$1" pin="9"/>
-<wire x1="167.64" y1="121.92" x2="160.02" y2="121.92" width="0.1524" layer="91"/>
-</segment>
-</net>
-<net name="N$4" class="0">
-<segment>
-<pinref part="D3" gate="G$1" pin="A"/>
-<wire x1="167.64" y1="134.62" x2="165.1" y2="134.62" width="0.1524" layer="91"/>
-<wire x1="165.1" y1="134.62" x2="165.1" y2="127" width="0.1524" layer="91"/>
-<pinref part="TEENSY2" gate="G$1" pin="11"/>
-<wire x1="165.1" y1="127" x2="160.02" y2="127" width="0.1524" layer="91"/>
-</segment>
-</net>
-<net name="N$5" class="0">
-<segment>
-<pinref part="D1" gate="G$1" pin="A"/>
-<pinref part="F1" gate="G$1" pin="P$2"/>
-<wire x1="17.78" y1="71.12" x2="17.78" y2="68.58" width="0.1524" layer="91"/>
-</segment>
-</net>
-<net name="N$6" class="0">
-<segment>
-<pinref part="C2" gate="G$1" pin="1"/>
-<wire x1="68.58" y1="50.8" x2="68.58" y2="53.34" width="0.1524" layer="91"/>
-<pinref part="U1" gate="G$1" pin="OUT"/>
-<wire x1="60.96" y1="53.34" x2="68.58" y2="53.34" width="0.1524" layer="91"/>
-<pinref part="D2" gate="G$1" pin="A"/>
-<wire x1="68.58" y1="55.88" x2="68.58" y2="53.34" width="0.1524" layer="91"/>
-<junction x="68.58" y="53.34"/>
-</segment>
-</net>
+<wire x1="165.1" y1="119.38" x2="165.1" y2="129.54" width="0.1524" layer="91"/>
+<pinref part="TEENSY2" gate="G$1" pin="12"/>
+<wire x1="165.1" y1="129.54" x2="160.02" y2="129.54" width="0.1524" layer="91"/>
+</segment>
+</net>

Commit message: fixed ledissues
Parts:
- added R1, R2, R3, R4, R5: (no value), resistor:R-US_R0603
Connections:
- new net N$5: D1.C, R5.2
- new net N$6: D2.C, R4.2
- new net N$7: D3.C, R1.1
- new net N$8: D4.C, R2.1
- new net N$9: D5.C, R3.1
- net GND: now also R1.2, R2.2, R3.2, R4.1, R5.1; no longer D1.C, D2.C, D3.C, D4.C, D5.C
Other:
- moved on the sheet: D1
Changed lines of the file:
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@@
 <part name="SUPPLY8" library="SparkFun-Aesthetics" deviceset="VCC" device="" value="9V"/>
 <part name="GND12" library="SparkFun-Aesthetics" deviceset="GND" device=""/>
+<part name="R1" library="resistor" deviceset="R-US_" device="R0603"/>
+<part name="R2" library="resistor" deviceset="R-US_" device="R0603"/>
+<part name="R3" library="resistor" deviceset="R-US_" device="R0603"/>
+<part name="R4" library="resistor" deviceset="R-US_" device="R0603"/>
+<part name="R5" library="resistor" deviceset="R-US_" device="R0603"/>
 </parts>
 <sheets>
@@
 <instance part="SUPPLY7" gate="G$1" x="198.12" y="76.2"/>
 <instance part="F1" gate="G$1" x="17.78" y="63.5" rot="R90"/>
-<instance part="D1" gate="G$1" x="7.62" y="76.2"/>
+<instance part="D1" gate="G$1" x="7.62" y="99.06"/>
 <instance part="D2" gate="G$1" x="83.82" y="58.42"/>
 <instance part="D3" gate="G$1" x="170.18" y="134.62" rot="R90"/>
 <instance part="D4" gate="G$1" x="170.18" y="127" rot="R90"/>
 <instance part="D5" gate="G$1" x="170.18" y="119.38" rot="R90"/>
-<instance part="GND9" gate="1" x="180.34" y="114.3"/>
+<instance part="GND9" gate="1" x="193.04" y="114.3"/>
 <instance part="SUPPLY4" gate="G$1" x="68.58" y="55.88"/>
-<instance part="GND11" gate="1" x="83.82" y="45.72"/>
+<instance part="GND11" gate="1" x="83.82" y="35.56"/>
 <instance part="SUPPLY6" gate="G$1" x="83.82" y="66.04"/>
-<instance part="SUPPLY8" gate="G$1" x="7.62" y="81.28"/>
-<instance part="GND12" gate="1" x="7.62" y="66.04"/>
+<instance part="SUPPLY8" gate="G$1" x="7.62" y="104.14"/>
+<instance part="GND12" gate="1" x="7.62" y="76.2"/>
+<instance part="R1" gate="G$1" x="187.96" y="134.62"/>
+<instance part="R2" gate="G$1" x="187.96" y="127"/>
+<instance part="R3" gate="G$1" x="187.96" y="119.38"/>
+<instance part="R4" gate="G$1" x="83.82" y="45.72" rot="R90"/>
+<instance part="R5" gate="G$1" x="7.62" y="86.36" rot="R90"/>
 </instances>
 <busses>
@@
 </segment>
 <segment>
-<pinref part="D5" gate="G$1" pin="C"/>
+<pinref part="GND12" gate="1" pin="GND"/>
+<pinref part="R5" gate="G$1" pin="1"/>
+<wire x1="7.62" y1="78.74" x2="7.62" y2="81.28" width="0.1524" layer="91"/>
+</segment>
+<segment>
+<pinref part="GND11" gate="1" pin="GND"/>
+<pinref part="R4" gate="G$1" pin="1"/>
+<wire x1="83.82" y1="38.1" x2="83.82" y2="40.64" width="0.1524" layer="91"/>
+</segment>
+<segment>
+<pinref part="R1" gate="G$1" pin="2"/>
+<pinref part="R2" gate="G$1" pin="2"/>
+<wire x1="193.04" y1="134.62" x2="193.04" y2="127" width="0.1524" layer="91"/>
+<pinref part="R3" gate="G$1" pin="2"/>
+<wire x1="193.04" y1="127" x2="193.04" y2="119.38" width="0.1524" layer="91"/>
+<junction x="193.04" y="127"/>
 <pinref part="GND9" gate="1" pin="GND"/>
-<wire x1="175.26" y1="119.38" x2="180.34" y2="119.38" width="0.1524" layer="91"/>
-<wire x1="180.34" y1="119.38" x2="180.34" y2="116.84" width="0.1524" layer="91"/>
-<pinref part="D4" gate="G$1" pin="C"/>
-<wire x1="175.26" y1="127" x2="180.34" y2="127" width="0.1524" layer="91"/>
-<wire x1="180.34" y1="127" x2="180.34" y2="119.38" width="0.1524" layer="91"/>
-<junction x="180.34" y="119.38"/>
-<pinref part="D3" gate="G$1" pin="C"/>
-<wire x1="175.26" y1="134.62" x2="180.34" y2="134.62" width="0.1524" layer="91"/>
-<wire x1="180.34" y1="134.62" x2="180.34" y2="127" width="0.1524" layer="91"/>
-<junction x="180.34" y="127"/>
-</segment>
-<segment>
-<pinref part="D2" gate="G$1" pin="C"/>
-<pinref part="GND11" gate="1" pin="GND"/>
-<wire x1="83.82" y1="53.34" x2="83.82" y2="48.26" width="0.1524" layer="91"/>
-</segment>
-<segment>
-<pinref part="D1" gate="G$1" pin="C"/>
-<pinref part="GND12" gate="1" pin="GND"/>
-<wire x1="7.62" y1="71.12" x2="7.62" y2="68.58" width="0.1524" layer="91"/>
+<wire x1="193.04" y1="119.38" x2="193.04" y2="116.84" width="0.1524" layer="91"/>
+<junction x="193.04" y="119.38"/>
 </segment>
 </net>
@@
 <pinref part="D1" gate="G$1" pin="A"/>
 <pinref part="SUPPLY8" gate="G$1" pin="VCC"/>
-<wire x1="7.62" y1="78.74" x2="7.62" y2="81.28" width="0.1524" layer="91"/>
+<wire x1="7.62" y1="101.6" x2="7.62" y2="104.14" width="0.1524" layer="91"/>
 </segment>
 </net>
@@
 </segment>
 </net>
+<net name="N$5" class="0">
+<segment>
+<pinref part="R5" gate="G$1" pin="2"/>
+<pinref part="D1" gate="G$1" pin="C"/>
+<wire x1="7.62" y1="91.44" x2="7.62" y2="93.98" width="0.1524" layer="91"/>
+</segment>
+</net>
+<net name="N$6" class="0">
+<segment>
+<pinref part="R4" gate="G$1" pin="2"/>
+<pinref part="D2" gate="G$1" pin="C"/>
+<wire x1="83.82" y1="50.8" x2="83.82" y2="53.34" width="0.1524" layer="91"/>
+</segment>
+</net>
+<net name="N$7" class="0">
+<segment>
+<pinref part="D3" gate="G$1" pin="C"/>
+<wire x1="175.26" y1="134.62" x2="182.88" y2="134.62" width="0.1524" layer="91"/>
+<pinref part="R1" gate="G$1" pin="1"/>
+</segment>
+</net>
+<net name="N$8" class="0">
+<segment>
+<pinref part="D4" gate="G$1" pin="C"/>
+<wire x1="175.26" y1="127" x2="182.88" y2="127" width="0.1524" layer="91"/>
+<pinref part="R2" gate="G$1" pin="1"/>
+</segment>
+</net>
+<net name="N$9" class="0">
+<segment>
+<pinref part="D5" gate="G$1" pin="C"/>
+<wire x1="175.26" y1="119.38" x2="182.88" y2="119.38" width="0.1524" layer="91"/>
+<pinref part="R3" gate="G$1" pin="1"/>
+</segment>
+</net>
